File: hardware/Eyeliner_PCB_V3/Eyeliner_PCB_V3.kicad_sch (KiCad schematic)
At the start: 0 parts

Commit message: Initial board bringup for v3.0
Other:
- removed sheet Bottom_Board
Changed lines of the file:
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@@
-	)
-	(sheet
-		(at 97.79 93.98)
-		(size 60.96 36.83)
-		(exclude_from_sim no)
-		(in_bom yes)
-		(on_board yes)
-		(dnp no)
-		(fields_autoplaced yes)
-		(stroke
-			(width 0.1524)
-			(type solid)
-		)
-		(fill
-			(color 0 0 0 0)
-		)
-		(property "Sheetname" "Bottom_Board"
-			(at 97.79 93.2684 0)
-			(show_name no)
-			(do_not_autoplace no)
-			(effects
-				(font
-					(size 1.27 1.27)
-				)
-				(justify left bottom)
-			)
-		)
-		(property "Sheetfile" "Top_Board.kicad_sch"
-			(at 97.79 131.3946 0)
-			(show_name no)
-			(do_not_autoplace no)
-			(effects
-				(font
-					(size 1.27 1.27)
-				)
-				(justify left top)
-			)
-		)
-		(instances
-			(project "Eyeliner_PCB_V3"
-				(path "/0cbb3bbb-8297-40d4-b3a9-e92b3d8d375c"
-					(page "3")
-				)
-			)
-		)
 	)
 	(sheet
