File: hardware/Eyeliner_PCB_V3/Top_Board.kicad_sch (KiCad schematic)
At the start: 0 parts

Commit message: Initial board bringup for v3.0
Parts:
- added Batt1: VBat, MountingHole:MountingHole_3.2mm_M3_DIN965_Pad, symbol Mechanical:MountingHole_Pad
- added C1: C0603X5R500-105KNP-CT, Capacitor_SMD:C_0603_1608Metric, symbol Device:C
- added C10, C11, C12, C13, C14, C15, C16, C18, C5: 100 nF, Capacitor_SMD:C_0402_1005Metric, symbol PCB-V2-Symbols:C
- added C17: 1uF, Capacitor_SMD:C_0402_1005Metric, symbol PCB-V2-Symbols:C
- added C19: GMC21X7R104K35NT, Capacitor_SMD:C_1206_3216Metric, symbol Device:C
- added C2: 100nF, Capacitor_SMD:C_0402_1005Metric, symbol Device:C
- added C20: GMT31X7R225K50NT2, Capacitor_SMD:C_1206_3216Metric, symbol Device:C
- added C3: 16pF, Capacitor_SMD:C_0402_1005Metric, symbol Device:C
- added C4, C6, C7, C8, C9: GMT32X7R106K35NT1, Capacitor_SMD:C_1210_3225Metric, symbol Device:C
- added D1: SPHV15-01ETG, Diode_SMD:D_SOD-882, symbol Device:D_Zener
- added D2: STPS2L30A, Diode_SMD:D_SMA, symbol Device:D_Schottky
- added D3: SMAJ6.0A, Diode_SMD:D_SMA, symbol Diode:PTVS26VZ1USK
- added D4: RCLAMP03348P.U, RCLAMP03348P_U:TVS_RCLAMP03348P.U, symbol RCLAMP03348P.U:RCLAMP03348P.U
- added D5: SMAJ30A or SMAJ24A, Diode_SMD:D_SMA, symbol Diode:PTVS26VZ1USK
- added ESCs1: JST_SH_01x06, Connector_JST:JST_SH_SM06B-SRSS-TB_1x06-1MP_P1.00mm_Horizontal, symbol Connector:Conn_01x06_Pin
- added GND1: GND_ESCs, MountingHole:MountingHole_3.2mm_M3_DIN965_Pad, symbol Mechanical:MountingHole_Pad
- added HV1: HV_ESCs, MountingHole:MountingHole_3.2mm_M3_DIN965_Pad, symbol Mechanical:MountingHole_Pad
- added I2C1, Temps1: JST_SH_01x04, Connector_JST:JST_SH_SM04B-SRSS-TB_1x04-1MP_P1.00mm_Horizontal, symbol Connector:Conn_01x04_Pin
- added J1: S7121-42R, S7121-42R:HARWIN_S7121-42R, symbol S7121-42R:S7121-42R
- added J3: SMTSO2020CTJ, MountingHole:SMTSO2020_Switch, symbol Connector:Conn_Coaxial_Power
- added L1: SRP1038A-150M, Bourns_SRP1038A:IND_SRP1038A_BRN, symbol Device:L
- added LEDs1: Conn_01x03_Pin, Connector_JST:JST_SH_SM03B-SRSS-TB_1x03-1MP_P1.00mm_Horizontal, symbol Connector:Conn_01x03_Pin
- added Q1: BSS138, Package_TO_SOT_SMD:SOT-323_SC-70, symbol Transistor_FET:BSS138
- added Q2: IRFR9020PBF, Package_TO_SOT_SMD:TO-252-2, symbol Simulation_SPICE:PMOS
- added R1: 100k, Resistor_SMD:R_0402_1005Metric, symbol Device:R
- added R12, R13, R14, R15, R16, R17, R18, R21, R22, R23, R24, R25, R30, R31: 100, Resistor_SMD:R_0402_1005Metric, symbol Device:R
- added R19, R20, R5: 1k, Resistor_SMD:R_0402_1005Metric, symbol Device:R
- added R2: 32.4k, Resistor_SMD:R_0402_1005Metric, symbol Device:R
- added R26, R27, R28, R29, R9: 4.7k, Resistor_SMD:R_0402_1005Metric, symbol Device:R
- added R3: 20k, Resistor_SMD:R_0402_1005Metric, symbol Device:R
- added R4: 5.1k, Resistor_SMD:R_0402_1005Metric, symbol Device:R
- added R6: 22k, Resistor_SMD:R_0402_1005Metric, symbol Device:R
- added R7: 2k, Resistor_SMD:R_0402_1005Metric, symbol Device:R
- added R8: RC1206FR-07100RL, Resistor_SMD:R_1206_3216Metric, symbol Device:R
- added Receiver1: (no value), Stuff from Walnut:BetaFPV ELRS Lite, symbol PCB-V2-Symbols:BetaFPVELRS
- added U1: LM61440AANRJRR, LM61440:LM61440AASQRJRRQ1, symbol LM61440AANRJRR:LM61440AANRJRR
- added U2: XIAO-ESP32-S3-SMD, Seeed_Studio_XIAO_Series:XIAO-ESP32-S3-SMD_Minimal, symbol Seeed Studio XIAO Series Library:XIAO-ESP32-S3-SMD
- added U3: TMUX154ERSW, Package_DFN_QFN:UQFN-10_1.4x1.8mm_P0.4mm, symbol Analog_Switch:TMUX154ERSW
- added U4, U5: LSM6DSV320XTR, Package_LGA:LGA-14_3x2.5mm_P0.5mm_LayoutBorder3x4y, symbol PCB-V2-Symbols:LSM6DSV320XTR
- added U6: TMUX1204DQAR, Package_SON:USON-10_2.5x1.0mm_P0.5mm, symbol TMUX1204:TMUX1204DQAR
- added U7: RCLAMP3346P.TNT, RCLAMP3346P:SGP2708N7_SEM, symbol RCLAMP3346P:RCLAMP3346P.TNT
Connections:
- new net: LEDs1.2 (Pin_2), R21.1
- new net: Q1.3 (D), R20.2, R21.2
- new net: C3.2, R5.1
- new net: D1.2 (A), Q2.2 (G), R1.1
- new net: I2C1.3 (Pin_3), R30.1
- new net: J1.SH1 (SHIELD), R8.2
- new net: Batt1.1, J3.2 (Ext)
- new net: R13.1, U2.4 (D3)
- new net: R12.2, U2.5 (D4)
- new net: R16.1, Temps1.3 (Pin_3)
- new net: ESCs1.6 (Pin_6), R22.1
- new net: R15.1, Temps1.2 (Pin_2)
- new net: C2.1, L1.1, U1.10 (SW)
- new net: C2.2, U1.13 (RBOOT), U1.14 (CBOOT)
- new net: C1.2, U1.2 (VCC)
- new net: R2.2, U1.6 (RT)
- new net: I2C1.2 (Pin_2), R31.2
- new net: ESCs1.5 (Pin_5), R23.1
- new net: R17.1, Temps1.4 (Pin_4)
- new net: ESCs1.2 (Pin_2), R25.1
- new net: ESCs1.3 (Pin_3), R24.1
- new net Bias: C3.1, C4.1, D2.2 (A), L1.2, R3.2, U1.1 (BIAS_1), U1.15 (BIAS_2)
- new net Dshot1: D4.9, R23.2, U2.9 (D8)
- new net Dshot2: D4.8, R25.2, U2.10 (D9)
- new net ESC_Telem1: D4.1, R22.2, U2.19 (MTMS)
- new net ESC_Telem2: D4.2, R24.2, U2.20 (MTCK)
- new net FB: R3.1, R4.2, R5.2, U1.4 (FB)
- new net GND: C1.1, C10.2, C11.2, C12.2, C13.2, C14.2, C15.2, C16.2, C17.2, C18.2, C19.2, C20.2, C4.2, C5.2, C6.2, C7.2, C8.2, C9.2, D3.2 (A), D4.3, D5.2 (A), ESCs1.1 (Pin_1), ESCs1.4 (Pin_4), GND1.1, I2C1.1 (Pin_1), LEDs1.1 (Pin_1), R1.2, R18.1, R2.1, R4.1, R7.1, Receiver1.4 (GND), Temps1.1 (Pin_1), U1.11 (PGND2_1), U1.17 (PGND1_2), U1.18 (PGND2_2), U1.3 (AGND), U1.9 (PGND1_1), U2.13 (GND), U3.4 (GND), U3.8 (~{EN}), U4.10 (OCS_AUX), U4.11 (SDO_AUX), U4.2 (SDX), U4.3 (SCX), U4.6 (GND), U4.7 (GND), U5.1 (SDO/TA0), U5.10 (OCS_AUX), U5.11 (SDO_AUX), U5.2 (SDX), U5.3 (SCX), U5.6 (GND), U5.7 (GND), U6.3 (GND), U7.2
- new net I2C_Sel: U2.15 (MTDI), U3.10 (SEL)
- new net INT: R9.1, U2.3 (D2), U4.4 (INT1), U5.4 (INT1)
- new net LEDs: Q1.2 (S), R19.2, U2.16 (MTDO), U7.1
- new net NC_1: U1.16 (PGOOD_2), U1.5 (PGOOD_1)
- new net Receiver_RX: R12.1, Receiver1.1 (RX), U7.3
- new net Receiver_TX: R13.2, Receiver1.2 (TX), U7.6
- new net SCL: U2.2 (D1), U3.5 (B)
- new net SCL_Accel: R27.1, U3.1 (A0), U4.13 (SCL), U5.13 (SCL)
- new net SCL_Extra: R29.1, R31.1, U3.6 (B1), U7.5
- new net SDA: U2.1 (D0), U3.3 (A)
- new net SDA_Accel: R26.1, U3.7 (B0), U4.14 (SDA), U5.14 (SDA)
- new net SDA_Extra: R28.1, R30.2, U3.2 (A1), U7.4
- new net Temp1_1: D4.7, R15.2, U6.7 (S4)
- new net Temp2_1: D4.6, R16.2, U6.4 (S3)
- new net Temp3_1: D4.5, R17.2, U6.2 (S1)
- new net TempRef_1: D4.4, R18.2, U6.9 (S2)
- new net Temp_Sel1: U2.7 (D6), U6.1 (A0)
- new net Temp_Sel2: U2.8 (D7), U6.10 (A1)
- new net Temp_Sense: C16.1, R14.1, U2.11 (D10), U6.8 (D)
- new net VCC_3V3: C10.1, C11.1, C12.1, C13.1, C14.1, C15.1, Q1.1 (G), R14.2, R19.1, R26.2, R27.2, R28.2, R29.2, R9.2, U2.12 (3V3_OUT), U3.9 (VCC), U4.1 (SDO/TA0), U4.12 (CS), U4.5 (VDDIO), U4.8 (VDD), U5.12 (CS), U5.5 (VDDIO), U5.8 (VDD), U6.5 (EN), U6.6 (VDD)
- new net VCC_5V: C17.1, C18.1, D2.1 (K), D3.1 (K), I2C1.4 (Pin_4), LEDs1.3 (Pin_3), R20.1, Receiver1.3 (5V), U2.14 (VBUS)
- new net VCC_HV: C19.1, C20.1, C6.1, C7.1, C8.1, C9.1, D1.1 (K), D5.1 (K), HV1.1, Q2.3 (S), R6.2, U1.12 (VIN2), U1.7 (EN/SYNC), U1.8 (VIN1)
- new net VCC_NoProc: Q2.1 (D), R8.1
- new net VCC_NoProc_SW: J3.1 (In)
- new net Vbat_Sense: C5.1, R6.1, R7.2, U2.6 (D5), U7.7
- no-connect marks 0 -> 2
Other:
- note added: "Core Logic"
- note added: "Ext Connections"
- note added: "Note: INT pins on LSM6DSVs are push-pull by default, need to set PP_OD in the CTRL3 register on both parts before enabling interrupts"

Commit message: Working on v3.1 board respin
Connections:
- net GND: no longer I2C1.1 (Pin_1)
- net SCL_Accel: now also U3.7 (B0); no longer U3.1 (A0)
- net SDA_Accel: now also U3.1 (A0); no longer U3.7 (B0)
- net VCC_5V: no longer I2C1.4 (Pin_4)
- net at R30.1: no longer I2C1.3 (Pin_3)
- net at R31.2: no longer I2C1.2 (Pin_2)
Other:
- moved on the sheet: I2C1
Changed lines of the file:
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@@
 		)
 	)
-	(label "SCL_Accel"
-		(at 104.14 210.82 0)
-		(effects
-			(font
-				(size 1.27 1.27)
-			)
-			(justify left bottom)
-		)
-	)
 	(label "INT"
 		(at 140.97 210.82 180)
@@
 		)
 	)
+	(label "SCL_Accel"
+		(at 104.14 220.98 0)
+		(effects
+			(font
+				(size 1.27 1.27)
+			)
+			(justify left bottom)
+		)
+	)
 	(label "Temp_Sel2"
 		(at 271.78 38.1 0)
@@
 		)
 	)
+	(label "SDA_Accel"
+		(at 104.14 210.82 0)
+		(effects
+			(font
+				(size 1.27 1.27)
+			)
+			(justify left bottom)
+		)
+	)
 	(label "SDA_Extra"
 		(at 104.14 215.9 0)
@@
 		)
 	)
-	(label "SDA_Accel"
-		(at 104.14 220.98 0)
-		(effects
-			(font
-				(size 1.27 1.27)
-			)
-			(justify left bottom)
-		)
-	)
 	(label "Bias"
 		(at 100.33 45.72 0)
@@
 		(in_pos_files yes)
 		(dnp no)
-		(fields_autoplaced yes)
 		(property "Reference" "U3"
 			(at 91.0433 200.66 0)
@@
 		)
 		(property "Value" "TMUX154ERSW"
-			(at 91.0433 203.2 0)
+			(at 90.932 203.2 0)
 			(show_name no)
 			(do_not_autoplace no)
@@
 	(symbol
 		(lib_id "Connector:Conn_01x04_Pin")
-		(at 323.85 36.83 180)
+		(at 554.228 -130.81 180)
 		(unit 1)
 		(body_style 1)
@@
 		(fields_autoplaced yes)
 		(property "Reference" "I2C1"
-			(at 325.12 34.2899 0)
+			(at 555.498 -133.3501 0)
 			(show_name no)
 			(do_not_autoplace no)
@@
 		)
 		(property "Value" "JST_SH_01x04"
-			(at 325.12 36.8299 0)
+			(at 555.498 -130.8101 0)
 			(show_name no)
 			(do_not_autoplace no)
@@
 		)
 		(property "Footprint" "Connector_JST:JST_SH_SM04B-SRSS-TB_1x04-1MP_P1.00mm_Horizontal"
-			(at 323.85 36.83 0)
+			(at 554.228 -130.81 0)
 			(hide yes)
 			(show_name no)
@@
 		)
 		(property "Datasheet" ""
-			(at 323.85 36.83 0)
+			(at 554.228 -130.81 0)
 			(hide yes)
 			(show_name no)
@@
 		)
 		(property "Description" "Generic connector, single row, 01x04, script generated"
-			(at 323.85 36.83 0)
+			(at 554.228 -130.81 0)
 			(hide yes)
 			(show_name no)

Commit message: All basic board functionality working
Parts:
- removed C12, C13, C15, C5: 100 nF, Capacitor_SMD:C_0402_1005Metric, symbol PCB-V2-Symbols:C
- removed C4, C8, C9: GMT32X7R106K35NT1, Capacitor_SMD:C_1210_3225Metric, symbol Device:C
- removed D1: SPHV15-01ETG, Diode_SMD:D_SOD-882, symbol Device:D_Zener
- removed D4: RCLAMP03348P.U, RCLAMP03348P_U:TVS_RCLAMP03348P.U, symbol RCLAMP03348P.U:RCLAMP03348P.U
- removed LEDs1: Conn_01x03_Pin, Connector_JST:JST_SH_SM03B-SRSS-TB_1x03-1MP_P1.00mm_Horizontal, symbol Connector:Conn_01x03_Pin
- removed Q2: IRFR9020PBF, Package_TO_SOT_SMD:TO-252-2, symbol Simulation_SPICE:PMOS
- removed R1: 100k, Resistor_SMD:R_0402_1005Metric, symbol Device:R
- removed R15, R16, R21: 100, Resistor_SMD:R_0402_1005Metric, symbol Device:R
- removed R20: 1k, Resistor_SMD:R_0402_1005Metric, symbol Device:R
- removed R28, R29: 4.7k, Resistor_SMD:R_0402_1005Metric, symbol Device:R
- removed R7: 2k, Resistor_SMD:R_0402_1005Metric, symbol Device:R
- removed Temps1: JST_SH_01x04, Connector_JST:JST_SH_SM04B-SRSS-TB_1x04-1MP_P1.00mm_Horizontal, symbol Connector:Conn_01x04_Pin
- removed U3: TMUX154ERSW, Package_DFN_QFN:UQFN-10_1.4x1.8mm_P0.4mm, symbol Analog_Switch:TMUX154ERSW
- added C11, C12, C16, C17: MSASG32MSB5226MPNA01, Capacitor_SMD:C_1210_3225Metric, symbol Device:C
- added Conn_LEDs1: JST_SH_01x04, Connector_JST:JST_SH_SM04B-SRSS-TB_1x04-1MP_P1.00mm_Horizontal, symbol Connector:Conn_01x04_Pin
- added IC1: PCA9570GMH, PCA9570:PCA9570GMH, symbol PCA9570GMH:PCA9570GMH
- added IC2: 74AHCT2G125DC,125, 74AHCT2G125DC, 125:SOP50P310X100-8N, symbol 74AHCT2G125DC_125:74AHCT2G125DC,125
- added IR1, RTD_Onboard1: TestPoint_2Pole, Capacitor_SMD:C_0805_2012Metric, symbol Connector:TestPoint_2Pole
- added R12: 2k, Resistor_SMD:R_0402_1005Metric, symbol Device:R
- added R24: 10k, Resistor_SMD:R_0402_1005Metric, symbol Device:R
- added R5: 100, Resistor_SMD:R_0402_1005Metric, symbol Device:R
- added Temps1: JST_SH_01x03, Connector_JST:JST_SH_SM03B-SRSS-TB_1x03-1MP_P1.00mm_Horizontal, symbol Connector:Conn_01x03_Pin
- added U7: RCLAMP3346P.TNT, RCLAMP3346P:SGP2708N7_SEM, symbol RCLAMP3346P:RCLAMP3346P.TNT
- Batt1, GND1, HV1: footprint MountingHole:MountingHole_3.2mm_M3_DIN965_Pad -> MountingHole:MountingHole_2.2mm_M2_Pad_Via
- C2: renamed from C19; footprint Capacitor_SMD:C_1206_3216Metric -> Capacitor_SMD:C_0805_2012Metric
- C3: renamed from C7; value GMT32X7R106K35NT1 -> MSASG32MSB5226MPNA01
- C4: renamed from C20; value GMT31X7R225K50NT2 -> GCJ31CR71H225KA12L
- C5: renamed from C6; value GMT32X7R106K35NT1 -> MSASG32MSB5226MPNA01
- C6: renamed from C10; value 100 nF -> 470nF
- C8: renamed from C11; value 100 nF -> 100nF
- J1: value S7121-42R -> S7131-45R
- J2: renamed from J3; value SMTSO2020CTJ -> 4871; footprint MountingHole:SMTSO2020_Switch -> MountingHole:4871_Switch_Precharge
- Q1: footprint Package_TO_SOT_SMD:SOT-323_SC-70 -> Package_TO_SOT_SMD:TSOT-23
- R10: renamed from R27; value 4.7k -> 1k
- R11: renamed from R6; value 22k -> 20k
- R13: renamed from R26; value 4.7k -> 1k
- R14: value 100 -> 1k
- R19: value 1k -> 4.7k
- R4: renamed from R2; value 32.4k -> 30k
- U2: footprint Seeed_Studio_XIAO_Series:XIAO-ESP32-S3-SMD_Minimal -> Seeed_Studio_XIAO_Series:XIAO-ESP32-S3-SMD
- renumbered C3 to C10, C17 to C13, C18 to C14, C16 to C15, C2 to C7, C14 to C9, D5 to D1, D3 to D2, D2 to D3, R9 to R1, R31 to R15, R30 to R16, R13 to R2, R24 to R20, R25 to R21, R12 to R3, R8 to R6, R3 to R7, R4 to R8, R5 to R9, U4 to U3, U5 to U4, U6 to U5, U7 to U6
Connections:
- net SCL_Accel is gone; now on net SCL: R10.1, U3.13 (SCL), U4.13 (SCL)
- net SDA_Accel is gone; now on net SDA: R13.1, U3.14 (SDA), U4.14 (SDA)
- net VCC_NoProc is gone; now on net VCC_HV: R6.1
- net VCC_NoProc_SW is gone; now on net VCC_HV: J2.1 (In)
- net Bias: now also D2.1 (K)
- net ESC_Telem1: now also U2.8 (D7); no longer U2.19 (MTMS)
- net ESC_Telem2: now also U2.11 (D10); no longer U2.20 (MTCK)
- net GND: now also ESCs1.3 (Pin_3), I2C1.1 (Pin_1), R19.1, U2.25 (PAD), C11.2, C12.2, C16.2, C17.2, Conn_LEDs1.1 (Pin_1), IC1.4 (VSS), IC2.4 (GND), IC2.7 (~{2OE}), R12.1, R24.1, R5.1, RTD_Onboard1.2, Temps1.1 (Pin_1), U7.2; no longer ESCs1.1 (Pin_1), R18.1
- net LEDs: now also IC2.5 (2A); no longer Q1.2 (S), R19.2
- net Receiver_RX: now also U6.4; no longer U6.3
- net Receiver_TX: now also U6.5; no longer U6.6
- net SCL: now also R15.1, IC1.6 (SCL), IC2.2 (1A), U7.5
- net SDA: now also R16.2, IC1.7 (SDA), U7.4
- net Temp1_1: now also R18.2, U6.6
- net Temp2_1: now also R17.2, U6.3
- net TempRef_1: now also R19.2, U5.2 (S1); no longer R18.2, U5.9 (S2)
- net Temp_Sel1: now also IC1.2 (P1); no longer U2.7 (D6)
- net Temp_Sel2: now also IC1.3 (P2); no longer U2.8 (D7)
- net VCC_3V3: now also IC1.8 (VDD); no longer Q1.1 (G), R19.1
- net VCC_5V: now also I2C1.4 (Pin_4), C11.1, C12.1, C16.1, C17.1, Conn_LEDs1.4 (Pin_4), IC2.8 (VCC), IR1.1; no longer D2.1 (K)
- net Vbat_Sense: now also U2.5 (D4), R12.2; no longer U2.6 (D5)
- net at Q1.3 (D): now also IR1.2
- net at R16.1: now also I2C1.3 (Pin_3)
- net at R2.1: now also U2.7 (D6); no longer U2.4 (D3)
- net at R3.2: now also U2.6 (D5); no longer U2.5 (D4)
- net ESC_Telem1_Proc: now reaches ESCs1.6 (Pin_6), R22.1
- net ESC_Telem1_Proc: now also U7.1
- net at R15.2: now also I2C1.2 (Pin_2)
- net Dshot1_Proc: now reaches ESCs1.5 (Pin_5), R23.1
- net Dshot1_Proc: now also U7.7
- net at R17.1: now also Temps1.2 (Pin_2)
- net Dshot2_Proc: now reaches ESCs1.2 (Pin_2), R21.1
- net Dshot2_Proc: now also U7.6
- net ESC_Telem2_Proc: now reaches R20.1
- net ESC_Telem2_Proc: now also ESCs1.1 (Pin_1), U7.3; no longer ESCs1.3 (Pin_3)
- removed net I2C_Sel: U2.15 (MTDI)
- removed net SCL_Extra: R15.1, U6.5
- removed net SDA_Extra: R16.2, U6.4
- removed net Temp3_1: R17.2, U5.2 (S1)
- net Temp_Sense renamed Sense
- net Sense: now also U2.4 (D3); no longer U2.11 (D10)
- new net: R18.1, Temps1.3 (Pin_3)
- new net: Conn_LEDs1.2 (Pin_2), IC2.3 (2Y)
- new net: Conn_LEDs1.3 (Pin_3), IC2.6 (1Y), R24.2
- new net: RTD_Onboard1.1, U5.9 (S2)
- new net: IC1.5 (P3), Q1.1 (G)
- new net: Q1.2 (S), R5.2
- new net LEDs_EN: IC1.1 (P0), IC2.1 (~{1OE})
Other:
- note added: "Power Section"
- moved on the sheet: D1, D2, D3, ESCs1, I2C1, R11, R15, R16, R20, R21, R22, R23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
